File: tipjar.sch (KiCad schematic (older format))
At the start: 55 parts, among them CON1 AVR-ISP-6, IC1 ATTINY85-S, P1 CONN_MICRO_USB_B, P2 CONN_2, P3 CONN_3, P4 CONN_3, P5 CONN_2, Q1 TSM2302, Q10 PHOTO_NPN, Q11 PHOTO_NPN, Q2 TSM2301, Q3 TSM2301, Q4 2N2222, Q5 2N2222, Q6 2N2222, Q7 2N2222, Q8 2N2222, Q9 2N2222, SW1 SW_PUSH, SW2 SW_PUSH, U1 MCP73831T-2ACI/OT, U2 MIC5504-3.3YM5

Commit message: Add lithium battery for data retention
Parts:
- added BT1: CR2032, ~, symbol BATTERY
- added D2, D3: CDBER40, ~, symbol DIODESCH
- renumbered D2 to D4, D3 to D5, D4 to D6, Q4 to Q3, Q3 to Q4, R9 to R10, R10 to R8, R8 to R9
Connections:
- wire segments 168 -> 212
Other:
- note added: "memory\nbuffer\nbattery"
- moved on the sheet: Q3, R8

Commit message: First remote commit
Parts:
- removed C4: 10µF, ~, symbol CP
- removed D5, D6: LED, ~, symbol LED
- removed JP3: JUMPER, ~, symbol JUMPER
- removed Q10, Q11: PHOTO_NPN, symbol PHOTO_TRANSISTOR
- removed R4: 100, ~, symbol R
- added C4: 1µF, Capacitors_SMD:C_0805, symbol C
- added C6: 10µF, Capacitors_SMD:C_0805, symbol C
- added D2: PMEG6030EP, VIC:SOD-128, symbol DIODESCH
- added U3, U4: ON1120, on1120:ON1120, symbol ON1120
- BT1: footprint ~ -> Battery_Holders:Keystone_3034_1x20mm-CoinCell
- C1, C5: footprint ~ -> Capacitors_SMD:C_0805; symbol C -> C-RESCUE-tipjar
- C2: footprint (none) -> Capacitors_SMD:C_0603; symbol C -> C-RESCUE-tipjar
- C3: renamed from C7; footprint ~ -> Capacitors_SMD:CP_Elec_6.3x7.7; symbol CP -> CP-RESCUE-tipjar
- C7: renamed from C3; footprint ~ -> Capacitors_SMD:C_0805; symbol C -> C-RESCUE-tipjar
- C8: renamed from C6; footprint ~ -> Capacitors_SMD:C_0603; symbol C -> C-RESCUE-tipjar
- C9: renamed from C8; footprint ~ -> Capacitors_SMD:C_0603; symbol C -> C-RESCUE-tipjar
- CON1: footprint AVR-ISP-6 -> Pin_Headers:Pin_Header_Straight_2x03_Pitch2.54mm
- D1: footprint ~ -> LEDs:LED_0603; symbol LED -> LED-RESCUE-tipjar
- D3: renamed from D2; value CDBER40 -> PMEG6030EP; footprint ~ -> VIC:SOD-128
- D4: renamed from D3; value CDBER40 -> PMEG6030EP; footprint ~ -> VIC:SOD-128
- D5: renamed from D4; footprint ~ -> LEDs:LED_0603; symbol LED -> LED-RESCUE-tipjar
- IC1: footprint SO8-200 -> Microcontrollers_ATTINY85-20SU:SOIC127P798X216-8N
- JP1: footprint ~ -> Pin_Headers:Pin_Header_Straight_1x02_Pitch2.54mm
- JP2: footprint ~ -> Pin_Headers:Pin_Header_Straight_1x03_Pitch2.54mm
- L1: renamed from L2; footprint ~ -> Inductors_SMD:L_12x12mm_h8mm
- L2: renamed from L1; footprint ~ -> Inductors_SMD:L_12x12mm_h8mm
- P1: footprint MODULE -> VIC:MICRO-B_USB
- P2: renamed from P5; footprint ~ -> Pin_Headers:Pin_Header_Straight_1x02_Pitch2.54mm
- P3: renamed from P2; footprint ~ -> Connectors_JST:JST_XH_B02B-XH-A_02x2.50mm_Straight
- P4: renamed from P3; footprint ~ -> Pin_Headers:Pin_Header_Straight_1x03_Pitch2.54mm
- P5: renamed from P4; footprint ~ -> Pin_Headers:Pin_Header_Straight_1x03_Pitch2.54mm
- Q1: renamed from Q2; footprint ~ -> TO_SOT_Packages_SMD:SOT-23
- Q2: renamed from Q1; footprint ~ -> TO_SOT_Packages_SMD:SOT-23
- Q3, Q4, Q6, Q7, Q8, Q9: footprint ~ -> TO_SOT_Packages_SMD:SOT-23
- Q5: footprint (none) -> TO_SOT_Packages_SMD:SOT-23
- R1, R2, R3, R8: footprint ~ -> Resistors_SMD:R_0603; symbol R -> R-RESCUE-tipjar
- R10: renamed from R11; value 1k2 -> 3k3; footprint ~ -> Resistors_SMD:R_0603; symbol R -> R-RESCUE-tipjar
- R11: renamed from R12; footprint ~ -> Resistors_SMD:R_0603; symbol R -> R-RESCUE-tipjar
- R12: renamed from R13; footprint ~ -> Resistors_SMD:R_0603; symbol R -> R-RESCUE-tipjar
- R13: renamed from R14; footprint (none) -> Resistors_SMD:R_0603; symbol R -> R-RESCUE-tipjar
- R14: renamed from R15; footprint ~ -> Resistors_SMD:R_0603; symbol R -> R-RESCUE-tipjar
- R15: renamed from R16; footprint ~ -> Resistors_SMD:R_0603; symbol R -> R-RESCUE-tipjar
- R4: renamed from R5; footprint ~ -> Resistors_SMD:R_0603; symbol R -> R-RESCUE-tipjar
- R5: renamed from R6; footprint ~ -> Resistors_SMD:R_0603; symbol R -> R-RESCUE-tipjar
- R6: renamed from R7; footprint ~ -> Resistors_SMD:R_0603; symbol R -> R-RESCUE-tipjar
- R7: renamed from R9; footprint ~ -> Resistors_SMD:R_0805_HandSoldering; symbol R -> R-RESCUE-tipjar
- R9: renamed from R10; footprint (none) -> Resistors_SMD:R_0603; symbol R -> R-RESCUE-tipjar
- SW1, SW2: footprint ~ -> Buttons_Switches_SMD:SW_SPST_EVQPE1
- U1: footprint Housings_SOT-23_SOT-143_TSOT-6:SOT-23-5 -> TO_SOT_Packages_SMD:SOT-23-5
- U2: footprint MODULE -> TO_SOT_Packages_SMD:SOT-23-5
Connections:
- wire segments 212 -> 173
Other:
- note added: "470 nF is enough (nF = ms)"
- note added: "Add Fuse!"
- note added: "Fast\nCharge\n500mA"
- note removed: "2 x OS25B10"
- note removed: "Fast\nCharge"
- note removed: "Power Source"
- moved on the sheet: C3, C5, C7, C8, C9, D5, JP2, L1, L2, P2, P3, P5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
